File: pcb/VEML3328-I2C-Sensor.kicad_pcb (KiCad board)
At the start: 2 copper layers, 18 x 26 mm, 11 parts, among them J1 Conn_01x04_Socket, J2 Conn_01x04_Pin, J3 Conn_01x04_Socket

Commit message: add pinout names
Other:
- board text added: "SCL SDA VCC GND"
